Commit message: updated lower and upper

File: genesis/assets/urdf/aliengo/urdf/aliengo.urdf (robot description, URDF)
Before this commit: robot aliengo, 18 links, 17 joints
Joints:
- joint FL_thigh_joint: limit effort=35.278 velocity=20 -> lower=-1.57 upper=3.49 effort=35.278 velocity=20
- joint FR_thigh_joint: limit effort=35.278 velocity=20 -> lower=-1.57 upper=3.49 effort=35.278 velocity=20
- joint RL_thigh_joint: limit effort=35.278 velocity=20 -> lower=-1.57 upper=3.49 effort=35.278 velocity=20
- joint RR_thigh_joint: limit effort=35.278 velocity=20 -> lower=-1.57 upper=3.49 effort=35.278 velocity=20
