Commit message: updated terrain and legged env for curriculum

File: genesis/assets/urdf/plane/custom_plane.urdf (robot description, URDF)
Before this commit: robot plane, 29 links, 28 joints
Links:
- link box_max_bottom: geometry collision box size=10.0 0.3 0.2; visual box size=10.0 0.3 0.2
- link box_max_left: geometry collision box size=0.3 10.0 0.2; visual box size=0.3 10.0 0.2
- link box_max_right: geometry collision box size=0.3 10.0 0.2; visual box size=0.3 10.0 0.2
- link box_max_top: geometry collision box size=10.0 0.3 0.2; visual box size=10.0 0.3 0.2
- link box_outer_bottom: geometry collision box size=8.0 0.3 0.15; visual box size=8.0 0.3 0.15
- link box_outer_left: geometry collision box size=0.3 8.0 0.15; visual box size=0.3 8.0 0.15
- link box_outer_right: geometry collision box size=0.3 8.0 0.15; visual box size=0.3 8.0 0.15
- link box_outer_top: geometry collision box size=8.0 0.3 0.15; visual box size=8.0 0.3 0.15

Commit message: updated go2 xml

File: genesis/assets/urdf/plane/custom_plane.urdf (robot description, URDF)
Before this commit: robot plane, 29 links, 28 joints
Links:
- removed link box_inner_bottom
- removed link box_inner_left
- removed link box_inner_right
- removed link box_inner_top
- removed link box_max_bottom
- removed link box_max_left
- removed link box_max_right
- removed link box_max_top
- removed link box_outer_bottom
- removed link box_outer_left
- removed link box_outer_right
- removed link box_outer_top
- added link box_down1_bottom; collision box size=13.8 0.3 0.15; visual box size=13.8 0.3 0.15
- added link box_down1_left; collision box size=0.3 13.8 0.15; visual box size=0.3 13.8 0.15
- added link box_down1_right; collision box size=0.3 13.8 0.15; visual box size=0.3 13.8 0.15
- added link box_down1_top; collision box size=13.8 0.3 0.15; visual box size=13.8 0.3 0.15
- added link box_down2_bottom; collision box size=14.4 0.3 0.15; visual box size=14.4 0.3 0.15
- added link box_down2_left; collision box size=0.3 14.4 0.15; visual box size=0.3 14.4 0.15
- added link box_down2_right; collision box size=0.3 14.4 0.15; visual box size=0.3 14.4 0.15
- added link box_down2_top; collision box size=14.4 0.3 0.15; visual box size=14.4 0.3 0.15
- added link box_down3_bottom; collision box size=15.0 0.3 0.15; visual box size=15.0 0.3 0.15
- added link box_down3_left; collision box size=0.3 15.0 0.15; visual box size=0.3 15.0 0.15
- added link box_down3_right; collision box size=0.3 15.0 0.15; visual box size=0.3 15.0 0.15
- added link box_down3_top; collision box size=15.0 0.3 0.15; visual box size=15.0 0.3 0.15
- added link box_inner1_bottom; collision box size=4.0 0.2 0.05; visual box size=4.0 0.2 0.05
- added link box_inner1_left; collision box size=0.2 4.0 0.05; visual box size=0.2 4.0 0.05
- added link box_inner1_right; collision box size=0.2 4.0 0.05; visual box size=0.2 4.0 0.05
- added link box_inner1_top; collision box size=4.0 0.2 0.05; visual box size=4.0 0.2 0.05
- added link box_inner2_bottom; collision box size=4.4 0.20 0.05; visual box size=4.4 0.20 0.05
- added link box_inner2_left; collision box size=0.20 4.4 0.05; visual box size=0.20 4.4 0.05
- added link box_inner2_right; collision box size=0.20 4.4 0.05; visual box size=0.20 4.4 0.05
- added link box_inner2_top; collision box size=4.4 0.20 0.05; visual box size=4.4 0.20 0.05
- added link box_inner3_bottom; collision box size=4.8 0.20 0.05; visual box size=4.8 0.20 0.05
- added link box_inner3_left; collision box size=0.20 4.8 0.05; visual box size=0.20 4.8 0.05
- added link box_inner3_right; collision box size=0.20 4.8 0.05; visual box size=0.20 4.8 0.05
- added link box_inner3_top; collision box size=4.8 0.20 0.05; visual box size=4.8 0.20 0.05
- added link box_outer1_bottom; collision box size=9.0 0.2 0.1; visual box size=9.0 0.2 0.1
- added link box_outer1_left; collision box size=0.2 9.0 0.1; visual box size=0.2 9.0 0.1
- added link box_outer1_right; collision box size=0.2 9.0 0.1; visual box size=0.2 9.0 0.1
- added link box_outer1_top; collision box size=9.0 0.2 0.1; visual box size=9.0 0.2 0.1
- added link box_outer2_bottom; collision box size=9.4 0.2 0.1; visual box size=9.4 0.2 0.1
- added link box_outer2_left; collision box size=0.2 9.4 0.1; visual box size=0.2 9.4 0.1
- added link box_outer2_right; collision box size=0.2 9.4 0.1; visual box size=0.2 9.4 0.1
- added link box_outer2_top; collision box size=9.4 0.2 0.1; visual box size=9.4 0.2 0.1
- added link box_outer3_bottom; collision box size=9.8 0.2 0.1; visual box size=9.8 0.2 0.1
- added link box_outer3_left; collision box size=0.2 9.8 0.1; visual box size=0.2 9.8 0.1
- added link box_outer3_right; collision box size=0.2 9.8 0.1; visual box size=0.2 9.8 0.1
- added link box_outer3_top; collision box size=9.8 0.2 0.1; visual box size=9.8 0.2 0.1
- added link box_stair4_bottom; collision box size=17.0 0.3 0.20; visual box size=17.0 0.3 0.20
- added link box_stair4_left; collision box size=0.3 17.0 0.20; visual box size=0.3 17.0 0.20
- added link box_stair4_right; collision box size=0.3 17.0 0.20; visual box size=0.3 17.0 0.20
- added link box_stair4_top; collision box size=17.0 0.3 0.20; visual box size=17.0 0.3 0.20
- added link box_stair5_bottom; collision box size=17.6 0.3 0.20; visual box size=17.6 0.3 0.20
- added link box_stair5_left; collision box size=0.3 17.6 0.20; visual box size=0.3 17.6 0.20
- added link box_stair5_right; collision box size=0.3 17.6 0.20; visual box size=0.3 17.6 0.20
- added link box_stair5_top; collision box size=17.6 0.3 0.20; visual box size=17.6 0.3 0.20
- added link box_stair6_bottom; collision box size=18.2 0.3 0.20; visual box size=18.2 0.3 0.20
- added link box_stair6_left; collision box size=0.3 18.2 0.20; visual box size=0.3 18.2 0.20
- added link box_stair6_right; collision box size=0.3 18.2 0.20; visual box size=0.3 18.2 0.20
- added link box_stair6_top; collision box size=18.2 0.3 0.20; visual box size=18.2 0.3 0.20
- added link box_stair_descend1_bottom; collision box size=18.8 0.3 0.20; visual box size=18.8 0.3 0.20
- added link box_stair_descend1_left; collision box size=0.3 18.8 0.20; visual box size=0.3 18.8 0.20
- added link box_stair_descend1_right; collision box size=0.3 18.8 0.20; visual box size=0.3 18.8 0.20
- added link box_stair_descend1_top; collision box size=18.8 0.3 0.20; visual box size=18.8 0.3 0.20
- added link box_stair_descend2_bottom; collision box size=19.4 0.3 0.20; visual box size=19.4 0.3 0.20
- added link box_stair_descend2_left; collision box size=0.3 19.4 0.20; visual box size=0.3 19.4 0.20
- added link box_stair_descend2_right; collision box size=0.3 19.4 0.20; visual box size=0.3 19.4 0.20
- added link box_stair_descend2_top; collision box size=19.4 0.3 0.20; visual box size=19.4 0.3 0.20
- added link box_stair_descend3_bottom; collision box size=20.0 0.3 0.20; visual box size=20.0 0.3 0.20
- added link box_stair_descend3_left; collision box size=0.3 20.0 0.20; visual box size=0.3 20.0 0.20
- added link box_stair_descend3_right; collision box size=0.3 20.0 0.20; visual box size=0.3 20.0 0.20
- added link box_stair_descend3_top; collision box size=20.0 0.3 0.20; visual box size=20.0 0.3 0.20
- link box_bottom: geometry collision box size=6.8 0.15 0.1; visual box size=6.8 0.15 0.1
- link box_left: geometry collision box size=0.15 6.8 0.1; visual box size=0.15 6.8 0.1
- link box_right: geometry collision box size=0.15 6.8 0.1; visual box size=0.15 6.8 0.1
- link box_stair1_bottom: geometry collision box size=12.0 0.3 0.15; visual box size=12.0 0.3 0.15
- link box_stair1_left: geometry collision box size=0.3 12.0 0.15; visual box size=0.3 12.0 0.15
- link box_stair1_right: geometry collision box size=0.3 12.0 0.15; visual box size=0.3 12.0 0.15
- link box_stair1_top: geometry collision box size=12.0 0.3 0.15; visual box size=12.0 0.3 0.15
- link box_stair2_bottom: geometry collision box size=12.6 0.3 0.15; visual box size=12.6 0.3 0.15
- link box_stair2_left: geometry collision box size=0.3 12.6 0.15; visual box size=0.3 12.6 0.15
- link box_stair2_right: geometry collision box size=0.3 12.6 0.15; visual box size=0.3 12.6 0.15
- link box_stair2_top: geometry collision box size=12.6 0.3 0.15; visual box size=12.6 0.3 0.15
- link box_stair3_bottom: geometry collision box size=13.2 0.3 0.15; visual box size=13.2 0.3 0.15
- link box_stair3_left: geometry collision box size=0.3 13.2 0.15; visual box size=0.3 13.2 0.15
- link box_stair3_right: geometry collision box size=0.3 13.2 0.15; visual box size=0.3 13.2 0.15
- link box_stair3_top: geometry collision box size=13.2 0.3 0.15; visual box size=13.2 0.3 0.15
- link box_top: geometry collision box size=6.8 0.15 0.1; visual box size=6.8 0.15 0.1
Joints:
- removed joint box_max_bottom
- removed joint box_max_left
- removed joint box_max_right
- removed joint box_max_top
- removed joint joint_inner_bottom
- removed joint joint_inner_left
- removed joint joint_inner_right
- removed joint joint_inner_top
- removed joint joint_outer_bottom
- removed joint joint_outer_left
- removed joint joint_outer_right
- removed joint joint_outer_top
- added joint box_down1_bottom: type fixed, parent planeLink, child box_down1_bottom, origin xyz=0 0 0
- added joint box_down1_left: type fixed, parent planeLink, child box_down1_left, origin xyz=0 0 0
- added joint box_down1_right: type fixed, parent planeLink, child box_down1_right, origin xyz=0 0 0
- added joint box_down1_top: type fixed, parent planeLink, child box_down1_top, origin xyz=0 0 0
- added joint box_down2_bottom: type fixed, parent planeLink, child box_down2_bottom, origin xyz=0 0 0
- added joint box_down2_left: type fixed, parent planeLink, child box_down2_left, origin xyz=0 0 0
- added joint box_down2_right: type fixed, parent planeLink, child box_down2_right, origin xyz=0 0 0
- added joint box_down2_top: type fixed, parent planeLink, child box_down2_top, origin xyz=0 0 0
- added joint box_down3_bottom: type fixed, parent planeLink, child box_down3_bottom, origin xyz=0 0 0
- added joint box_down3_left: type fixed, parent planeLink, child box_down3_left, origin xyz=0 0 0
- added joint box_down3_right: type fixed, parent planeLink, child box_down3_right, origin xyz=0 0 0
- added joint box_down3_top: type fixed, parent planeLink, child box_down3_top, origin xyz=0 0 0
- added joint box_stair4_bottom: type fixed, parent planeLink, child box_stair4_bottom, origin xyz=0 0 0
- added joint box_stair4_left: type fixed, parent planeLink, child box_stair4_left, origin xyz=0 0 0
- added joint box_stair4_right: type fixed, parent planeLink, child box_stair4_right, origin xyz=0 0 0
- added joint box_stair4_top: type fixed, parent planeLink, child box_stair4_top, origin xyz=0 0 0
- added joint box_stair5_bottom: type fixed, parent planeLink, child box_stair5_bottom, origin xyz=0 0 0
- added joint box_stair5_left: type fixed, parent planeLink, child box_stair5_left, origin xyz=0 0 0
- added joint box_stair5_right: type fixed, parent planeLink, child box_stair5_right, origin xyz=0 0 0
- added joint box_stair5_top: type fixed, parent planeLink, child box_stair5_top, origin xyz=0 0 0
- added joint box_stair6_bottom: type fixed, parent planeLink, child box_stair6_bottom, origin xyz=0 0 0
- added joint box_stair6_left: type fixed, parent planeLink, child box_stair6_left, origin xyz=0 0 0
- added joint box_stair6_right: type fixed, parent planeLink, child box_stair6_right, origin xyz=0 0 0
- added joint box_stair6_top: type fixed, parent planeLink, child box_stair6_top, origin xyz=0 0 0
- added joint box_stair_descend1_bottom: type fixed, parent planeLink, child box_stair_descend1_bottom, origin xyz=0 0 0
- added joint box_stair_descend1_left: type fixed, parent planeLink, child box_stair_descend1_left, origin xyz=0 0 0
- added joint box_stair_descend1_right: type fixed, parent planeLink, child box_stair_descend1_right, origin xyz=0 0 0
- added joint box_stair_descend1_top: type fixed, parent planeLink, child box_stair_descend1_top, origin xyz=0 0 0
- added joint box_stair_descend2_bottom: type fixed, parent planeLink, child box_stair_descend2_bottom, origin xyz=0 0 0
- added joint box_stair_descend2_left: type fixed, parent planeLink, child box_stair_descend2_left, origin xyz=0 0 0
- added joint box_stair_descend2_right: type fixed, parent planeLink, child box_stair_descend2_right, origin xyz=0 0 0
- added joint box_stair_descend2_top: type fixed, parent planeLink, child box_stair_descend2_top, origin xyz=0 0 0
- added joint box_stair_descend3_bottom: type fixed, parent planeLink, child box_stair_descend3_bottom, origin xyz=0 0 0
- added joint box_stair_descend3_left: type fixed, parent planeLink, child box_stair_descend3_left, origin xyz=0 0 0
- added joint box_stair_descend3_right: type fixed, parent planeLink, child box_stair_descend3_right, origin xyz=0 0 0
- added joint box_stair_descend3_top: type fixed, parent planeLink, child box_stair_descend3_top, origin xyz=0 0 0
- added joint joint_inner1_bottom: type fixed, parent planeLink, child box_inner1_bottom, origin xyz=0 0 0
- added joint joint_inner1_left: type fixed, parent planeLink, child box_inner1_left, origin xyz=0 0 0
- added joint joint_inner1_right: type fixed, parent planeLink, child box_inner1_right, origin xyz=0 0 0
- added joint joint_inner1_top: type fixed, parent planeLink, child box_inner1_top, origin xyz=0 0 0
- added joint joint_inner2_bottom: type fixed, parent planeLink, child box_inner2_bottom, origin xyz=0 0 0
- added joint joint_inner2_left: type fixed, parent planeLink, child box_inner2_left, origin xyz=0 0 0
- added joint joint_inner2_right: type fixed, parent planeLink, child box_inner2_right, origin xyz=0 0 0
- added joint joint_inner2_top: type fixed, parent planeLink, child box_inner2_top, origin xyz=0 0 0
- added joint joint_inner3_bottom: type fixed, parent planeLink, child box_inner3_bottom, origin xyz=0 0 0
- added joint joint_inner3_left: type fixed, parent planeLink, child box_inner3_left, origin xyz=0 0 0
- added joint joint_inner3_right: type fixed, parent planeLink, child box_inner3_right, origin xyz=0 0 0
- added joint joint_inner3_top: type fixed, parent planeLink, child box_inner3_top, origin xyz=0 0 0
- added joint joint_outer1_bottom: type fixed, parent planeLink, child box_outer1_bottom, origin xyz=0 0 0
- added joint joint_outer1_left: type fixed, parent planeLink, child box_outer1_left, origin xyz=0 0 0
- added joint joint_outer1_right: type fixed, parent planeLink, child box_outer1_right, origin xyz=0 0 0
- added joint joint_outer1_top: type fixed, parent planeLink, child box_outer1_top, origin xyz=0 0 0
- added joint joint_outer2_bottom: type fixed, parent planeLink, child box_outer2_bottom, origin xyz=0 0 0
- added joint joint_outer2_left: type fixed, parent planeLink, child box_outer2_left, origin xyz=0 0 0
- added joint joint_outer2_right: type fixed, parent planeLink, child box_outer2_right, origin xyz=0 0 0
- added joint joint_outer2_top: type fixed, parent planeLink, child box_outer2_top, origin xyz=0 0 0
- added joint joint_outer3_bottom: type fixed, parent planeLink, child box_outer3_bottom, origin xyz=0 0 0
- added joint joint_outer3_left: type fixed, parent planeLink, child box_outer3_left, origin xyz=0 0 0
- added joint joint_outer3_right: type fixed, parent planeLink, child box_outer3_right, origin xyz=0 0 0
- added joint joint_outer3_top: type fixed, parent planeLink, child box_outer3_top, origin xyz=0 0 0

Commit message: fixed a logical mistake

File: genesis/assets/urdf/plane/custom_plane.urdf (robot description, URDF)
Before this commit: robot plane, 77 links, 76 joints
Links:
- link box_outer3_bottom: geometry collision box size=9.8 0.5 0.1; visual box size=9.8 0.5 0.1
- link box_outer3_left: geometry collision box size=0.5 9.8 0.1; visual box size=0.5 9.8 0.1
- link box_outer3_right: geometry collision box size=0.5 9.8 0.1; visual box size=0.5 9.8 0.1
- link box_outer3_top: geometry collision box size=9.8 0.5 0.1; visual box size=9.8 0.5 0.1
